Commit message: feat(description): expand urdf model to multi-joint industrial manipulator arm

File: src/inspector_description/urdf/inspector_arm.urdf.xacro (robot description, xacro)
@@ -1,20 +1,28 @@
 <?xml version="1.0"?>
 <robot xmlns:xacro="http://www.ros.org/wiki/xacro" name="industrial_inspector">
+  <!-- Materials -->
+  <material name="dark_grey"><color rgba="0.2 0.2 0.2 1.0"/></material>
+  <material name="orange"><color rgba="1.0 0.5 0.0 1.0"/></material>
+  <material name="light_grey"><color rgba="0.7 0.7 0.7 1.0"/></material>
+  <material name="blue"><color rgba="0.0 0.4 0.8 1.0"/></material>
+  <!-- World Link -->
+  <link name="world"/>
+  <joint name="world_joint" type="fixed">
+    <parent link="world"/>
+    <child link="base_link"/>
+    <origin xyz="0 0 0" rpy="0 0 0"/>
+  </joint>
+  <!-- Base Link -->
   <link name="base_link">
     <visual>
-      <geometry>
-        <cylinder length="0.1" radius="0.2"/>
-      </geometry>
-      <material name="dark_grey">
-        <color rgba="0.2 0.2 0.2 1.0"/>
-      </material>
+      <geometry><cylinder length="0.1" radius="0.2"/></geometry>
+      <material name="dark_grey"/>
     </visual>
     <collision>
-      <geometry>
-        <cylinder length="0.1" radius="0.2"/>
-      </geometry>
+      <geometry><cylinder length="0.1" radius="0.2"/></geometry>
     </collision>
   </link>
-  <joint name="shoulder_joint" type="revolute">
+  <!-- Joint 1: Base Rotation -->
+  <joint name="joint_1" type="revolute">
     <parent link="base_link"/>
     <child link="shoulder_link"/>
@@ -25,11 +33,52 @@
   <link name="shoulder_link">
     <visual>
-      <geometry>
-        <cylinder length="0.4" radius="0.08"/>
-      </geometry>
+      <geometry><cylinder length="0.2" radius="0.1"/></geometry>
+      <origin xyz="0 0 0.1" rpy="0 0 0"/>
+      <material name="orange"/>
+    </visual>
+  </link>
+  <!-- Joint 2: Upper Arm Pitch -->
+  <joint name="joint_2" type="revolute">
+    <parent link="shoulder_link"/>
+    <child link="upper_arm_link"/>
+    <origin xyz="0 0 0.2" rpy="0 0 0"/>
+    <axis xyz="0 1 0"/>
+    <limit lower="-1.57" upper="1.57" effort="100" velocity="1.0"/>
+  </joint>
+  <link name="upper_arm_link">
+    <visual>
+      <geometry><box size="0.08 0.08 0.5"/></geometry>
+      <origin xyz="0 0 0.25" rpy="0 0 0"/>
+      <material name="light_grey"/>
+    </visual>
+  </link>
+  <!-- Joint 3: Forearm Pitch -->
+  <joint name="joint_3" type="revolute">
+    <parent link="upper_arm_link"/>
+    <child link="forearm_link"/>
+    <origin xyz="0 0 0.5" rpy="0 0 0"/>
+    <axis xyz="0 1 0"/>
+    <limit lower="-1.57" upper="1.57" effort="100" velocity="1.0"/>
+  </joint>
+  <link name="forearm_link">
+    <visual>
+      <geometry><box size="0.06 0.06 0.4"/></geometry>
       <origin xyz="0 0 0.2" rpy="0 0 0"/>
-      <material name="orange">
-        <color rgba="1.0 0.5 0.0 1.0"/>
-      </material>
+      <material name="orange"/>
+    </visual>
+  </link>
+  <!-- Joint 4: Wrist Roll / Tool Flange -->
+  <joint name="joint_4" type="revolute">
+    <parent link="forearm_link"/>
+    <child link="wrist_link"/>
+    <origin xyz="0 0 0.4" rpy="0 0 0"/>
+    <axis xyz="0 0 1"/>
+    <limit lower="-3.14" upper="3.14" effort="50" velocity="2.0"/>
+  </joint>
+  <link name="wrist_link">
+    <visual>
+      <geometry><cylinder length="0.08" radius="0.05"/></geometry>
+      <origin xyz="0 0 0.04" rpy="0 0 0"/>
+      <material name="blue"/>
     </visual>
   </link>

Commit message: feat(bringup): add inertial properties to urdf and setup gazebo simulation bringup package

File: src/inspector_description/urdf/inspector_arm.urdf.xacro (robot description, xacro)
@@ -1,10 +1,8 @@
 <?xml version="1.0"?>
 <robot xmlns:xacro="http://www.ros.org/wiki/xacro" name="industrial_inspector">
-  <!-- Materials -->
   <material name="dark_grey"><color rgba="0.2 0.2 0.2 1.0"/></material>
   <material name="orange"><color rgba="1.0 0.5 0.0 1.0"/></material>
   <material name="light_grey"><color rgba="0.7 0.7 0.7 1.0"/></material>
   <material name="blue"><color rgba="0.0 0.4 0.8 1.0"/></material>
-  <!-- World Link -->
   <link name="world"/>
   <joint name="world_joint" type="fixed">
@@ -22,6 +20,11 @@
       <geometry><cylinder length="0.1" radius="0.2"/></geometry>
     </collision>
+    <inertial>
+      <mass value="5.0"/>
+      <origin xyz="0 0 0" rpy="0 0 0"/>
+      <inertia ixx="0.05" ixy="0" ixz="0" iyy="0.05" iyz="0" izz="0.1"/>
+    </inertial>
   </link>
-  <!-- Joint 1: Base Rotation -->
+  <!-- Joint 1 -->
   <joint name="joint_1" type="revolute">
     <parent link="base_link"/>
@@ -37,6 +40,15 @@
       <material name="orange"/>
     </visual>
+    <collision>
+      <geometry><cylinder length="0.2" radius="0.1"/></geometry>
+      <origin xyz="0 0 0.1" rpy="0 0 0"/>
+    </collision>
+    <inertial>
+      <mass value="2.0"/>
+      <origin xyz="0 0 0.1" rpy="0 0 0"/>
+      <inertia ixx="0.01" ixy="0" ixz="0" iyy="0.01" iyz="0" izz="0.01"/>
+    </inertial>
   </link>
-  <!-- Joint 2: Upper Arm Pitch -->
+  <!-- Joint 2 -->
   <joint name="joint_2" type="revolute">
     <parent link="shoulder_link"/>
@@ -52,34 +64,13 @@
       <material name="light_grey"/>
     </visual>
-  </link>
-  <!-- Joint 3: Forearm Pitch -->
-  <joint name="joint_3" type="revolute">
-    <parent link="upper_arm_link"/>
-    <child link="forearm_link"/>
-    <origin xyz="0 0 0.5" rpy="0 0 0"/>
-    <axis xyz="0 1 0"/>
-    <limit lower="-1.57" upper="1.57" effort="100" velocity="1.0"/>
-  </joint>
-  <link name="forearm_link">
-    <visual>
-      <geometry><box size="0.06 0.06 0.4"/></geometry>
-      <origin xyz="0 0 0.2" rpy="0 0 0"/>
-      <material name="orange"/>
-    </visual>
-  </link>
-  <!-- Joint 4: Wrist Roll / Tool Flange -->
-  <joint name="joint_4" type="revolute">
-    <parent link="forearm_link"/>
-    <child link="wrist_link"/>
-    <origin xyz="0 0 0.4" rpy="0 0 0"/>
-    <axis xyz="0 0 1"/>
-    <limit lower="-3.14" upper="3.14" effort="50" velocity="2.0"/>
-  </joint>
-  <link name="wrist_link">
-    <visual>
-      <geometry><cylinder length="0.08" radius="0.05"/></geometry>
-      <origin xyz="0 0 0.04" rpy="0 0 0"/>
-      <material name="blue"/>
-    </visual>
+    <collision>
+      <geometry><box size="0.08 0.08 0.5"/></geometry>
+      <origin xyz="0 0 0.25" rpy="0 0 0"/>
+    </collision>
+    <inertial>
+      <mass value="1.5"/>
+      <origin xyz="0 0 0.25" rpy="0 0 0"/>
+      <inertia ixx="0.03" ixy="0" ixz="0" iyy="0.03" iyz="0" izz="0.005"/>
+    </inertial>
   </link>
 </robot>

Commit message: feat(control): integrate ros2_control configuration and gazebo ros2_control plugin

File: src/inspector_description/urdf/inspector_arm.urdf.xacro (robot description, xacro)
@@ -50,27 +50,19 @@
     </inertial>
   </link>
-  <!-- Joint 2 -->
-  <joint name="joint_2" type="revolute">
-    <parent link="shoulder_link"/>
-    <child link="upper_arm_link"/>
-    <origin xyz="0 0 0.2" rpy="0 0 0"/>
-    <axis xyz="0 1 0"/>
-    <limit lower="-1.57" upper="1.57" effort="100" velocity="1.0"/>
-  </joint>
-  <link name="upper_arm_link">
-    <visual>
-      <geometry><box size="0.08 0.08 0.5"/></geometry>
-      <origin xyz="0 0 0.25" rpy="0 0 0"/>
-      <material name="light_grey"/>
-    </visual>
-    <collision>
-      <geometry><box size="0.08 0.08 0.5"/></geometry>
-      <origin xyz="0 0 0.25" rpy="0 0 0"/>
-    </collision>
-    <inertial>
-      <mass value="1.5"/>
-      <origin xyz="0 0 0.25" rpy="0 0 0"/>
-      <inertia ixx="0.03" ixy="0" ixz="0" iyy="0.03" iyz="0" izz="0.005"/>
-    </inertial>
-  </link>
+  <!-- ros2_control Hardware Interface Definition -->
+  <ros2_control name="GazeboSimSystem" type="system">
+    <hardware>
+      <plugin>gz_ros2_control/GazeboSimSystem</plugin>
+    </hardware>
+    <joint name="joint_1">
+      <command_interface name="position"/>
+      <state_interface name="position"/>
+      <state_interface name="velocity"/>
+    </joint>
+  </ros2_control>
+  <gazebo>
+    <plugin filename="gz_ros2_control-system" name="gz_ros2_control::GazeboSimROS2ControlPlugin">
+      <parameters>$(find inspector_bringup)/config/controllers.yaml</parameters>
+    </plugin>
+  </gazebo>
 </robot>

Commit message: feat(arm+control): extend to 4-DOF chain and spawn ros2_control controllers in sim
- Add joint_2/3/4 links + ros2_control interfaces to match controllers.yaml
- Update SRDF planning group and collision pairs for 4-joint arm
- Spawn joint_state_broadcaster and arm_controller after robot appears in Gazebo
- Add missing controller_manager exec_depend

File: src/inspector_description/urdf/inspector_arm.urdf.xacro (robot description, xacro)
@@ -50,4 +50,76 @@
     </inertial>
   </link>
+  <!-- Joint 2 -->
+  <joint name="joint_2" type="revolute">
+    <parent link="shoulder_link"/>
+    <child link="upper_arm_link"/>
+    <origin xyz="0 0 0.2" rpy="0 0 0"/>
+    <axis xyz="0 1 0"/>
+    <limit lower="-1.57" upper="1.57" effort="100" velocity="1.0"/>
+  </joint>
+  <link name="upper_arm_link">
+    <visual>
+      <geometry><cylinder length="0.3" radius="0.08"/></geometry>
+      <origin xyz="0 0 0.15" rpy="0 0 0"/>
+      <material name="light_grey"/>
+    </visual>
+    <collision>
+      <geometry><cylinder length="0.3" radius="0.08"/></geometry>
+      <origin xyz="0 0 0.15" rpy="0 0 0"/>
+    </collision>
+    <inertial>
+      <mass value="1.5"/>
+      <origin xyz="0 0 0.15" rpy="0 0 0"/>
+      <inertia ixx="0.01" ixy="0" ixz="0" iyy="0.01" iyz="0" izz="0.005"/>
+    </inertial>
+  </link>
+  <!-- Joint 3 -->
+  <joint name="joint_3" type="revolute">
+    <parent link="upper_arm_link"/>
+    <child link="forearm_link"/>
+    <origin xyz="0 0 0.3" rpy="0 0 0"/>
+    <axis xyz="0 1 0"/>
+    <limit lower="-1.57" upper="1.57" effort="80" velocity="1.0"/>
+  </joint>
+  <link name="forearm_link">
+    <visual>
+      <geometry><cylinder length="0.25" radius="0.06"/></geometry>
+      <origin xyz="0 0 0.125" rpy="0 0 0"/>
+      <material name="blue"/>
+    </visual>
+    <collision>
+      <geometry><cylinder length="0.25" radius="0.06"/></geometry>
+      <origin xyz="0 0 0.125" rpy="0 0 0"/>
+    </collision>
+    <inertial>
+      <mass value="1.0"/>
+      <origin xyz="0 0 0.125" rpy="0 0 0"/>
+      <inertia ixx="0.005" ixy="0" ixz="0" iyy="0.005" iyz="0" izz="0.002"/>
+    </inertial>
+  </link>
+  <!-- Joint 4 (wrist) -->
+  <joint name="joint_4" type="revolute">
+    <parent link="forearm_link"/>
+    <child link="wrist_link"/>
+    <origin xyz="0 0 0.25" rpy="0 0 0"/>
+    <axis xyz="0 0 1"/>
+    <limit lower="-3.14" upper="3.14" effort="40" velocity="1.5"/>
+  </joint>
+  <link name="wrist_link">
+    <visual>
+      <geometry><cylinder length="0.08" radius="0.05"/></geometry>
+      <origin xyz="0 0 0.04" rpy="0 0 0"/>
+      <material name="dark_grey"/>
+    </visual>
+    <collision>
+      <geometry><cylinder length="0.08" radius="0.05"/></geometry>
+      <origin xyz="0 0 0.04" rpy="0 0 0"/>
+    </collision>
+    <inertial>
+      <mass value="0.5"/>
+      <origin xyz="0 0 0.04" rpy="0 0 0"/>
+      <inertia ixx="0.001" ixy="0" ixz="0" iyy="0.001" iyz="0" izz="0.001"/>
+    </inertial>
+  </link>
   <!-- ros2_control Hardware Interface Definition -->
   <ros2_control name="GazeboSimSystem" type="system">
@@ -56,4 +128,19 @@
     </hardware>
     <joint name="joint_1">
+      <command_interface name="position"/>
+      <state_interface name="position"/>
+      <state_interface name="velocity"/>
+    </joint>
+    <joint name="joint_2">
+      <command_interface name="position"/>
+      <state_interface name="position"/>
+      <state_interface name="velocity"/>
+    </joint>
+    <joint name="joint_3">
+      <command_interface name="position"/>
+      <state_interface name="position"/>
+      <state_interface name="velocity"/>
+    </joint>
+    <joint name="joint_4">
       <command_interface name="position"/>
       <state_interface name="position"/>

Commit message: Fix ros2_control/gz_ros2_control ABI crash, resolve xacro plugin path bug, complete 4-joint MoveIt config, add working full_system launch with OMPL fix, update README

File: src/inspector_description/urdf/inspector_arm.urdf.xacro (robot description, xacro)
@@ -1,4 +1,5 @@
 <?xml version="1.0"?>
 <robot xmlns:xacro="http://www.ros.org/wiki/xacro" name="industrial_inspector">
+  <xacro:arg name="controllers_config" default=""/>
   <material name="dark_grey"><color rgba="0.2 0.2 0.2 1.0"/></material>
   <material name="orange"><color rgba="1.0 0.5 0.0 1.0"/></material>
@@ -50,4 +51,76 @@
     </inertial>
   </link>
+  <!-- Joint 2 -->
+  <joint name="joint_2" type="revolute">
+    <parent link="shoulder_link"/>
+    <child link="upper_arm_link"/>
+    <origin xyz="0 0 0.2" rpy="0 0 0"/>
+    <axis xyz="0 1 0"/>
+    <limit lower="-1.57" upper="1.57" effort="100" velocity="1.0"/>
+  </joint>
+  <link name="upper_arm_link">
+    <visual>
+      <geometry><cylinder length="0.3" radius="0.08"/></geometry>
+      <origin xyz="0 0 0.15" rpy="0 0 0"/>
+      <material name="light_grey"/>
+    </visual>
+    <collision>
+      <geometry><cylinder length="0.3" radius="0.08"/></geometry>
+      <origin xyz="0 0 0.15" rpy="0 0 0"/>
+    </collision>
+    <inertial>
+      <mass value="1.5"/>
+      <origin xyz="0 0 0.15" rpy="0 0 0"/>
+      <inertia ixx="0.01" ixy="0" ixz="0" iyy="0.01" iyz="0" izz="0.005"/>
+    </inertial>
+  </link>
+  <!-- Joint 3 -->
+  <joint name="joint_3" type="revolute">
+    <parent link="upper_arm_link"/>
+    <child link="forearm_link"/>
+    <origin xyz="0 0 0.3" rpy="0 0 0"/>
+    <axis xyz="0 1 0"/>
+    <limit lower="-1.57" upper="1.57" effort="80" velocity="1.0"/>
+  </joint>
+  <link name="forearm_link">
+    <visual>
+      <geometry><cylinder length="0.25" radius="0.06"/></geometry>
+      <origin xyz="0 0 0.125" rpy="0 0 0"/>
+      <material name="blue"/>
+    </visual>
+    <collision>
+      <geometry><cylinder length="0.25" radius="0.06"/></geometry>
+      <origin xyz="0 0 0.125" rpy="0 0 0"/>
+    </collision>
+    <inertial>
+      <mass value="1.0"/>
+      <origin xyz="0 0 0.125" rpy="0 0 0"/>
+      <inertia ixx="0.005" ixy="0" ixz="0" iyy="0.005" iyz="0" izz="0.002"/>
+    </inertial>
+  </link>
+  <!-- Joint 4 (wrist) -->
+  <joint name="joint_4" type="revolute">
+    <parent link="forearm_link"/>
+    <child link="wrist_link"/>
+    <origin xyz="0 0 0.25" rpy="0 0 0"/>
+    <axis xyz="0 0 1"/>
+    <limit lower="-3.14" upper="3.14" effort="40" velocity="1.5"/>
+  </joint>
+  <link name="wrist_link">
+    <visual>
+      <geometry><cylinder length="0.08" radius="0.05"/></geometry>
+      <origin xyz="0 0 0.04" rpy="0 0 0"/>
+      <material name="dark_grey"/>
+    </visual>
+    <collision>
+      <geometry><cylinder length="0.08" radius="0.05"/></geometry>
+      <origin xyz="0 0 0.04" rpy="0 0 0"/>
+    </collision>
+    <inertial>
+      <mass value="0.5"/>
+      <origin xyz="0 0 0.04" rpy="0 0 0"/>
+      <inertia ixx="0.001" ixy="0" ixz="0" iyy="0.001" iyz="0" izz="0.001"/>
+    </inertial>
+  </link>
   <!-- ros2_control Hardware Interface Definition -->
   <ros2_control name="GazeboSimSystem" type="system">
@@ -60,8 +133,23 @@
       <state_interface name="velocity"/>
     </joint>
+    <joint name="joint_2">
+      <command_interface name="position"/>
+      <state_interface name="position"/>
+      <state_interface name="velocity"/>
+    </joint>
+    <joint name="joint_3">
+      <command_interface name="position"/>
+      <state_interface name="position"/>
+      <state_interface name="velocity"/>
+    </joint>
+    <joint name="joint_4">
+      <command_interface name="position"/>
+      <state_interface name="position"/>
+      <state_interface name="velocity"/>
+    </joint>
   </ros2_control>
   <gazebo>
     <plugin filename="gz_ros2_control-system" name="gz_ros2_control::GazeboSimROS2ControlPlugin">
-      <parameters>$(find inspector_bringup)/config/controllers.yaml</parameters>
+      <parameters>$(arg controllers_config)</parameters>
     </plugin>
   </gazebo>

Commit message: feat(description): add parallel-jaw gripper, widen elbow limit, add gripper controller

File: src/inspector_description/urdf/inspector_arm.urdf.xacro (robot description, xacro)
@@ -81,5 +81,5 @@
     <origin xyz="0 0 0.3" rpy="0 0 0"/>
     <axis xyz="0 1 0"/>
-    <limit lower="-1.57" upper="1.57" effort="80" velocity="1.0"/>
+    <limit lower="-2.4" upper="2.4" effort="80" velocity="1.0"/>
   </joint>
   <link name="forearm_link">
@@ -123,4 +123,81 @@
     </inertial>
   </link>
+  <!-- ===================== Parallel-jaw gripper ===================== -->
+  <joint name="gripper_palm_joint" type="fixed">
+    <parent link="wrist_link"/>
+    <child link="gripper_palm"/>
+    <origin xyz="0 0 0.08" rpy="0 0 0"/>
+  </joint>
+  <link name="gripper_palm">
+    <visual>
+      <geometry><box size="0.04 0.12 0.02"/></geometry>
+      <origin xyz="0 0 0.01" rpy="0 0 0"/>
+      <material name="dark_grey"/>
+    </visual>
+    <collision>
+      <geometry><box size="0.04 0.12 0.02"/></geometry>
+      <origin xyz="0 0 0.01" rpy="0 0 0"/>
+    </collision>
+    <inertial>
+      <mass value="0.1"/>
+      <origin xyz="0 0 0.01" rpy="0 0 0"/>
+      <inertia ixx="0.0002" ixy="0" ixz="0" iyy="0.0001" iyz="0" izz="0.0002"/>
+    </inertial>
+  </link>
+  <joint name="finger_left_joint" type="prismatic">
+    <parent link="gripper_palm"/>
+    <child link="finger_left_link"/>
+    <origin xyz="0 0.025 0.02" rpy="0 0 0"/>
+    <axis xyz="0 1 0"/>
+    <limit lower="-0.01" upper="0.03" effort="30" velocity="0.1"/>
+  </joint>
+  <link name="finger_left_link">
+    <visual>
+      <geometry><box size="0.03 0.012 0.06"/></geometry>
+      <origin xyz="0 0.006 0.03" rpy="0 0 0"/>
+      <material name="orange"/>
+    </visual>
+    <collision>
+      <geometry><box size="0.03 0.012 0.06"/></geometry>
+      <origin xyz="0 0.006 0.03" rpy="0 0 0"/>
+    </collision>
+    <inertial>
+      <mass value="0.05"/>
+      <origin xyz="0 0.006 0.03" rpy="0 0 0"/>
+      <inertia ixx="0.00002" ixy="0" ixz="0" iyy="0.00002" iyz="0" izz="0.00001"/>
+    </inertial>
+  </link>
+  <joint name="finger_right_joint" type="prismatic">
+    <parent link="gripper_palm"/>
+    <child link="finger_right_link"/>
+    <origin xyz="0 -0.025 0.02" rpy="0 0 0"/>
+    <axis xyz="0 -1 0"/>
+    <limit lower="-0.01" upper="0.03" effort="30" velocity="0.1"/>
+  </joint>
+  <link name="finger_right_link">
+    <visual>
+      <geometry><box size="0.03 0.012 0.06"/></geometry>
+      <origin xyz="0 -0.006 0.03" rpy="0 0 0"/>
+      <material name="orange"/>
+    </visual>
+    <collision>
+      <geometry><box size="0.03 0.012 0.06"/></geometry>
+      <origin xyz="0 -0.006 0.03" rpy="0 0 0"/>
+    </collision>
+    <inertial>
+      <mass value="0.05"/>
+      <origin xyz="0 -0.006 0.03" rpy="0 0 0"/>
+      <inertia ixx="0.00002" ixy="0" ixz="0" iyy="0.00002" iyz="0" izz="0.00001"/>
+    </inertial>
+  </link>
+  <!-- Tool centre point: 0.13 m beyond the wrist joint -->
+  <joint name="tool_center_joint" type="fixed">
+    <parent link="gripper_palm"/>
+    <child link="tool_center"/>
+    <origin xyz="0 0 0.05" rpy="0 0 0"/>
+  </joint>
+  <link name="tool_center"/>
+  <gazebo reference="finger_left_link"><mu1>1.5</mu1><mu2>1.5</mu2></gazebo>
+  <gazebo reference="finger_right_link"><mu1>1.5</mu1><mu2>1.5</mu2></gazebo>
   <!-- ros2_control Hardware Interface Definition -->
   <ros2_control name="GazeboSimSystem" type="system">
@@ -144,4 +221,14 @@
     </joint>
     <joint name="joint_4">
+      <command_interface name="position"/>
+      <state_interface name="position"/>
+      <state_interface name="velocity"/>
+    </joint>
+    <joint name="finger_left_joint">
+      <command_interface name="position"/>
+      <state_interface name="position"/>
+      <state_interface name="velocity"/>
+    </joint>
+    <joint name="finger_right_joint">
       <command_interface name="position"/>
       <state_interface name="position"/>
